File: hardware/ControlFPGAConfig.kicad_sch (KiCad schematic)
At the start: 29 parts, among them J5 JTAG_CONFIG, SW2 SW_DIP_x03, U10 SN74LVC2G17DCKRE4, U4 XC7S25-1CSGA225C, U8 IS25LP064A-JLLE, U9 SN74LVC2G17DCKRE4

Commit message: Update hardware design and include board logo
Sync the saved schematics, PCB, project settings, and referenced custom
libraries with the updated design. Include the LOGO footprint and register
it in the project footprint table. The board now contains 524 footprints.

Keep unused source libraries, autosaves, backups, analysis outputs, and
manufacturing files out of the import. Point BOM exports to the existing
ignored production directory instead of a workstation-specific location.

Validation with KiCad 9.0.1:
- Netlist export succeeds and referenced custom libraries resolve.
- DRC: 0 errors, 40 warnings, 0 unconnected items, 0 schematic mismatches.
- ERC: 27 errors and 71 warnings, identical to the source design.

The pre-existing missing JTAG 3D model (87831-1420.stp) is not supplied by
the source project and remains unresolved.
Parts:
- D5: value G_LED -> B_LED; LCSC C5342733 -> C19171394
- R51: renamed from R50; LCSC C99782 -> C22548
- R52: renamed from R51; LCSC C99782 -> C22548
- R53: renamed from R52; LCSC C99782 -> C22548
- renumbered C189 to C193, C190 to C194, C191 to C195, R47 to R48, R48 to R49, R49 to R50, R53 to R54, R54 to R55, R55 to R56, R56 to R57, R57 to R58, R58 to R59, R59 to R60, R60 to R61, R61 to R62, R62 to R63, R63 to R64, U9 to U10, U10 to U11, U4 to U5, U8 to U9
Connections:
- net C_LED_4: no longer names the net of R64.1, U5.K11 (IO_L3P_T0_DQS_PUDC_B_14)
