File: hardware/ControlFPGAPeripheral.kicad_sch (KiCad schematic)
At the start: 23 parts, among them SW10 SW_DIP_x08, SW8 SW_MEC_5E, SW9 SW_MEC_5E

Commit message: Update hardware design and include board logo
Sync the saved schematics, PCB, project settings, and referenced custom
libraries with the updated design. Include the LOGO footprint and register
it in the project footprint table. The board now contains 524 footprints.

Keep unused source libraries, autosaves, backups, analysis outputs, and
manufacturing files out of the import. Point BOM exports to the existing
ignored production directory instead of a workstation-specific location.

Validation with KiCad 9.0.1:
- Netlist export succeeds and referenced custom libraries resolve.
- DRC: 0 errors, 40 warnings, 0 unconnected items, 0 schematic mismatches.
- ERC: 27 errors and 71 warnings, identical to the source design.

The pre-existing missing JTAG 3D model (87831-1420.stp) is not supplied by
the source project and remains unresolved.
Parts:
- renumbered R72 to R73, R73 to R74, R74 to R75, R75 to R76, R76 to R77, R77 to R78, R78 to R79, R79 to R80, R80 to R81, R81 to R82
Changed lines of the file:
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@@
 		(on_board yes)
 		(dnp no)
-		(property "Reference" "R81"
+		(property "Reference" "R82"
 			(at 57.658 108.204 0)
 			(effects
@@
 			(project "shamiko"
 				(path "/3bdb682e-16f1-4662-9b00-b0c9070eb240/f0c15594-86ae-4f77-9d8c-bcbad84ec943"
-					(reference "R81")
+					(reference "R82")
 					(unit 1)
 				)
@@
 		(dnp no)
 		(fields_autoplaced yes)
-		(property "Reference" "R73"
+		(property "Reference" "R74"
 			(at 182.88 48.2599 0)
 			(effects
@@
 			(project "shamiko"
 				(path "/3bdb682e-16f1-4662-9b00-b0c9070eb240/f0c15594-86ae-4f77-9d8c-bcbad84ec943"
-					(reference "R73")
+					(reference "R74")
 					(unit 1)
 				)
@@
 		(dnp no)
 		(fields_autoplaced yes)
-		(property "Reference" "R75"
+		(property "Reference" "R76"
 			(at 208.28 48.2599 0)
 			(effects
@@
 			(project "shamiko"
 				(path "/3bdb682e-16f1-4662-9b00-b0c9070eb240/f0c15594-86ae-4f77-9d8c-bcbad84ec943"
-					(reference "R75")
+					(reference "R76")
 					(unit 1)
 				)
@@
 		(dnp no)
 		(fields_autoplaced yes)
-		(property "Reference" "#PWR0265"
+		(property "Reference" "#PWR0264"
 			(at 49.53 133.35 0)
 			(effects
@@
 			(project "shamiko"
 				(path "/3bdb682e-16f1-4662-9b00-b0c9070eb240/f0c15594-86ae-4f77-9d8c-bcbad84ec943"
-					(reference "#PWR0265")
+					(reference "#PWR0264")
 					(unit 1)
 				)
@@
 		(dnp no)
 		(fields_autoplaced yes)
-		(property "Reference" "R77"
+		(property "Reference" "R78"
 			(at 233.68 48.2599 0)
 			(effects
@@
 			(project "shamiko"
 				(path "/3bdb682e-16f1-4662-9b00-b0c9070eb240/f0c15594-86ae-4f77-9d8c-bcbad84ec943"
-					(reference "R77")
+					(reference "R78")
 					(unit 1)
 				)
@@
 		(dnp no)
 		(fields_autoplaced yes)
-		(property "Reference" "R72"
+		(property "Reference" "R73"
 			(at 170.18 48.2599 0)
 			(effects
@@
 			(project "shamiko"
 				(path "/3bdb682e-16f1-4662-9b00-b0c9070eb240/f0c15594-86ae-4f77-9d8c-bcbad84ec943"
-					(reference "R72")
+					(reference "R73")
 					(unit 1)
 				)
@@
 		(dnp no)
 		(fields_autoplaced yes)
-		(property "Reference" "R78"
+		(property "Reference" "R79"
 			(at 246.38 48.2599 0)
 			(effects
@@
 			(project "shamiko"
 				(path "/3bdb682e-16f1-4662-9b00-b0c9070eb240/f0c15594-86ae-4f77-9d8c-bcbad84ec943"
-					(reference "R78")
+					(reference "R79")
 					(unit 1)
 				)
@@
 		(dnp no)
 		(fields_autoplaced yes)
-		(property "Reference" "R74"
+		(property "Reference" "R75"
 			(at 195.58 48.2599 0)
 			(effects
@@
 			(project "shamiko"
 				(path "/3bdb682e-16f1-4662-9b00-b0c9070eb240/f0c15594-86ae-4f77-9d8c-bcbad84ec943"
-					(reference "R74")
+					(reference "R75")
 					(unit 1)
 				)
@@
 		(dnp no)
 		(fields_autoplaced yes)
-		(property "Reference" "R76"
+		(property "Reference" "R77"
 			(at 220.98 48.2599 0)
 			(effects
@@
 			(project "shamiko"
 				(path "/3bdb682e-16f1-4662-9b00-b0c9070eb240/f0c15594-86ae-4f77-9d8c-bcbad84ec943"
-					(reference "R76")
+					(reference "R77")
 					(unit 1)
 				)
@@
 		(on_board yes)
 		(dnp no)
-		(property "Reference" "R80"
+		(property "Reference" "R81"
 			(at 50.038 108.204 0)
 			(effects
@@
 			(project ""
 				(path "/3bdb682e-16f1-4662-9b00-b0c9070eb240/f0c15594-86ae-4f77-9d8c-bcbad84ec943"
-					(reference "R80")
+					(reference "R81")
 					(unit 1)
 				)
@@
 		(dnp no)
 		(fields_autoplaced yes)
-		(property "Reference" "R79"
+		(property "Reference" "R80"
 			(at 259.08 48.2599 0)
 			(effects
@@
 			(project "shamiko"
 				(path "/3bdb682e-16f1-4662-9b00-b0c9070eb240/f0c15594-86ae-4f77-9d8c-bcbad84ec943"
-					(reference "R79")
-					(unit 1)
-				)
+					(reference "R80")
+					(unit 1)
+				)
