File: hardware/ControlFPGASv.kicad_sch (KiCad schematic)
At the start: 22 parts, among them J11 SMA, J12 SMA, SW13 SW_MEC_5E, SW14 SW_MEC_5E, Y4 HCI 1532P-48.000KWVDT

Commit message: Update hardware design and include board logo
Sync the saved schematics, PCB, project settings, and referenced custom
libraries with the updated design. Include the LOGO footprint and register
it in the project footprint table. The board now contains 524 footprints.

Keep unused source libraries, autosaves, backups, analysis outputs, and
manufacturing files out of the import. Point BOM exports to the existing
ignored production directory instead of a workstation-specific location.

Validation with KiCad 9.0.1:
- Netlist export succeeds and referenced custom libraries resolve.
- DRC: 0 errors, 40 warnings, 0 unconnected items, 0 schematic mismatches.
- ERC: 27 errors and 71 warnings, identical to the source design.

The pre-existing missing JTAG 3D model (87831-1420.stp) is not supplied by
the source project and remains unresolved.
Parts:
- C257: renamed from C252; now not fitted
- R107: renamed from R104; LCSC C95204 -> C2906993
- R108: renamed from R105; LCSC C95204 -> C862232
- R109: renamed from R106; LCSC C95204 -> C105579
- Y4: value HCI 1532P-48.000KWVDT -> HCI 1532H-48.000GWVATS
- renumbered C247 to C252, C248 to C253, C249 to C254, C250 to C255, C251 to C256, C253 to C258, R100 to R103, R101 to R104, R102 to R105, R103 to R106
