File: hardware/ControllerFPGAHeader.kicad_sch (KiCad schematic)
At the start: 4 parts, among them J7 Conn_02x08

Commit message: Update hardware design and include board logo
Sync the saved schematics, PCB, project settings, and referenced custom
libraries with the updated design. Include the LOGO footprint and register
it in the project footprint table. The board now contains 524 footprints.

Keep unused source libraries, autosaves, backups, analysis outputs, and
manufacturing files out of the import. Point BOM exports to the existing
ignored production directory instead of a workstation-specific location.

Validation with KiCad 9.0.1:
- Netlist export succeeds and referenced custom libraries resolve.
- DRC: 0 errors, 40 warnings, 0 unconnected items, 0 schematic mismatches.
- ERC: 27 errors and 71 warnings, identical to the source design.

The pre-existing missing JTAG 3D model (87831-1420.stp) is not supplied by
the source project and remains unresolved.
Parts:
- C199: renamed from C195; footprint Capacitor_SMD:C_0603_1608Metric -> Capacitor_SMD:C_0805_2012Metric; LCSC C77386 -> C126592
- renumbered C196 to C200, C197 to C201
Changed lines of the file:
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@@
 		(dnp no)
 		(fields_autoplaced yes)
-		(property "Reference" "C197"
+		(property "Reference" "C201"
 			(at 226.06 78.7399 0)
 			(effects
@@
 			(project "shamiko"
 				(path "/3bdb682e-16f1-4662-9b00-b0c9070eb240/3f9015ba-1e1b-4181-8827-9de0bcfaf07f"
-					(reference "C197")
+					(reference "C201")
 					(unit 1)
 				)
@@
 		(dnp no)
 		(fields_autoplaced yes)
-		(property "Reference" "#PWR0262"
+		(property "Reference" "#PWR0261"
 			(at 222.25 107.95 0)
 			(effects
@@
 			(project "shamiko"
 				(path "/3bdb682e-16f1-4662-9b00-b0c9070eb240/3f9015ba-1e1b-4181-8827-9de0bcfaf07f"
-					(reference "#PWR0262")
+					(reference "#PWR0261")
 					(unit 1)
 				)
@@
 		(dnp no)
 		(fields_autoplaced yes)
-		(property "Reference" "C195"
+		(property "Reference" "C199"
 			(at 200.66 78.7399 0)
 			(effects
@@
 			)
 		)
-		(property "Footprint" "Capacitor_SMD:C_0603_1608Metric"
+		(property "Footprint" "Capacitor_SMD:C_0805_2012Metric"
 			(at 197.8152 83.82 0)
 			(effects
@@
 			)
 		)
-		(property "LCSC" "C77386 "
+		(property "LCSC" "C126592"
 			(at 196.85 80.01 0)
 			(effects
@@
 			(project "shamiko"
 				(path "/3bdb682e-16f1-4662-9b00-b0c9070eb240/3f9015ba-1e1b-4181-8827-9de0bcfaf07f"
-					(reference "C195")
+					(reference "C199")
 					(unit 1)
 				)
@@
 		(dnp no)
 		(fields_autoplaced yes)
-		(property "Reference" "#PWR0256"
+		(property "Reference" "#PWR0255"
 			(at 127 40.64 0)
 			(effects
@@
 			(project "shamiko"
 				(path "/3bdb682e-16f1-4662-9b00-b0c9070eb240/3f9015ba-1e1b-4181-8827-9de0bcfaf07f"
-					(reference "#PWR0256")
+					(reference "#PWR0255")
 					(unit 1)
 				)
@@
 		(dnp no)
 		(fields_autoplaced yes)
-		(property "Reference" "#PWR0257"
+		(property "Reference" "#PWR0256"
 			(at 196.85 62.23 0)
 			(effects
@@
 			(project "shamiko"
 				(path "/3bdb682e-16f1-4662-9b00-b0c9070eb240/3f9015ba-1e1b-4181-8827-9de0bcfaf07f"
-					(reference "#PWR0257")
+					(reference "#PWR0256")
 					(unit 1)
 				)
@@
 		(dnp no)
 		(fields_autoplaced yes)
-		(property "Reference" "#PWR0260"
+		(property "Reference" "#PWR0259"
 			(at 196.85 107.95 0)
 			(effects
@@
 			(project "shamiko"
 				(path "/3bdb682e-16f1-4662-9b00-b0c9070eb240/3f9015ba-1e1b-4181-8827-9de0bcfaf07f"
-					(reference "#PWR0260")
+					(reference "#PWR0259")
 					(unit 1)
 				)
@@
 		(dnp no)
 		(fields_autoplaced yes)
-		(property "Reference" "C196"
+		(property "Reference" "C200"
 			(at 213.36 78.7399 0)
 			(effects
@@
 			(project "shamiko"
 				(path "/3bdb682e-16f1-4662-9b00-b0c9070eb240/3f9015ba-1e1b-4181-8827-9de0bcfaf07f"
-					(reference "C196")
+					(reference "C200")
 					(unit 1)
 				)
@@
 		(dnp no)
 		(fields_autoplaced yes)
-		(property "Reference" "#PWR0259"
+		(property "Reference" "#PWR0258"
 			(at 139.7 106.68 0)
 			(effects
@@
 			(project "shamiko"
 				(path "/3bdb682e-16f1-4662-9b00-b0c9070eb240/3f9015ba-1e1b-4181-8827-9de0bcfaf07f"
-					(reference "#PWR0259")
+					(reference "#PWR0258")
 					(unit 1)
 				)
@@
 		(dnp no)
 		(fields_autoplaced yes)
-		(property "Reference" "#PWR0258"
+		(property "Reference" "#PWR0257"
 			(at 209.55 62.23 0)
 			(effects
@@
 			(project "shamiko"
 				(path "/3bdb682e-16f1-4662-9b00-b0c9070eb240/3f9015ba-1e1b-4181-8827-9de0bcfaf07f"
-					(reference "#PWR0258")
+					(reference "#PWR0257")
 					(unit 1)
 				)
@@
 		(dnp no)
 		(fields_autoplaced yes)
-		(property "Reference" "#PWR0255"
+		(property "Reference" "#PWR0254"
 			(at 120.65 40.64 0)
 			(effects
@@
 			(project "shamiko"
 				(path "/3bdb682e-16f1-4662-9b00-b0c9070eb240/3f9015ba-1e1b-4181-8827-9de0bcfaf07f"
-					(reference "#PWR0255")
+					(reference "#PWR0254")
 					(unit 1)
 				)
@@
 		(dnp no)
 		(fields_autoplaced yes)
-		(property "Reference" "#PWR0261"
+		(property "Reference" "#PWR0260"
 			(at 209.55 107.95 0)
 			(effects
@@
 			(project "shamiko"
 				(path "/3bdb682e-16f1-4662-9b00-b0c9070eb240/3f9015ba-1e1b-4181-8827-9de0bcfaf07f"
-					(reference "#PWR0261")
-					(unit 1)
-				)
+					(reference "#PWR0260")
+					(unit 1)
+				)
