File: hardware/ControllerFPGAPower.kicad_sch (KiCad schematic)
At the start: 47 parts, among them U4 XC7S25-1CSGA225C

Commit message: Update hardware design and include board logo
Sync the saved schematics, PCB, project settings, and referenced custom
libraries with the updated design. Include the LOGO footprint and register
it in the project footprint table. The board now contains 524 footprints.

Keep unused source libraries, autosaves, backups, analysis outputs, and
manufacturing files out of the import. Point BOM exports to the existing
ignored production directory instead of a workstation-specific location.

Validation with KiCad 9.0.1:
- Netlist export succeeds and referenced custom libraries resolve.
- DRC: 0 errors, 40 warnings, 0 unconnected items, 0 schematic mismatches.
- ERC: 27 errors and 71 warnings, identical to the source design.

The pre-existing missing JTAG 3D model (87831-1420.stp) is not supplied by
the source project and remains unresolved.
Parts:
- C147: renamed from C143; LCSC C90057 -> C90057
- C148: renamed from C144; LCSC C90057 -> C90057
- C154: renamed from C150; LCSC C90057 -> C90057
- C155: renamed from C151; LCSC C90057 -> C90057
- C161: renamed from C157; LCSC C90057 -> C90057
- C162: renamed from C158; LCSC C90057 -> C90057
- C168: renamed from C164; LCSC C90057 -> C90057
- C169: renamed from C165; LCSC C90057 -> C90057
- C170: renamed from C166; LCSC C90057 -> C90057
- C174: renamed from C170; LCSC C90057 -> C90057
- C175: renamed from C171; LCSC C90057 -> C90057
- C181: renamed from C177; LCSC C85973 -> C15195
- C182: renamed from C178; LCSC C90057 -> C90057
- C183: renamed from C179; LCSC C90057 -> C90057
- C188: renamed from C184; LCSC C90057 -> C90057
- renumbered C142 to C146, C145 to C149, C146 to C150, C147 to C151, C148 to C152, C149 to C153, C152 to C156, C153 to C157, C154 to C158, C155 to C159, C156 to C160, C159 to C163, C160 to C164, C161 to C165, C162 to C166, C163 to C167, C167 to C171, C168 to C172, C169 to C173, C172 to C176, C173 to C177, C174 to C178, C175 to C179, C176 to C180, C180 to C184, C181 to C185, C182 to C186, C183 to C187, C185 to C189, U4 to U5
