File: hardware/CurrentSensAmplifer.kicad_sch (KiCad schematic)
At the start: 27 parts, among them IC8 LT1763CS8-5#PBF, J13 SMA, U14 AD8000

Commit message: Update hardware design and include board logo
Sync the saved schematics, PCB, project settings, and referenced custom
libraries with the updated design. Include the LOGO footprint and register
it in the project footprint table. The board now contains 524 footprints.

Keep unused source libraries, autosaves, backups, analysis outputs, and
manufacturing files out of the import. Point BOM exports to the existing
ignored production directory instead of a workstation-specific location.

Validation with KiCad 9.0.1:
- Netlist export succeeds and referenced custom libraries resolve.
- DRC: 0 errors, 40 warnings, 0 unconnected items, 0 schematic mismatches.
- ERC: 27 errors and 71 warnings, identical to the source design.

The pre-existing missing JTAG 3D model (87831-1420.stp) is not supplied by
the source project and remains unresolved.
Parts:
- C259: renamed from C254; footprint Capacitor_SMD:C_0603_1608Metric -> Capacitor_SMD:C_0805_2012Metric; LCSC C77386 -> C126592
- C261: renamed from C256; LCSC C440198 -> C126586
- C265: renamed from C260; value 1000p -> 1n
- C266: renamed from C261; value 1000p -> 1n
- C273: renamed from C268; value 1000p -> 1n
- R117: renamed from R114; value 61.9 -> 62; LCSC C830425 -> C230313
- renumbered C255 to C260, C257 to C262, C258 to C263, C259 to C264, C262 to C267, C263 to C268, C264 to C269, C265 to C270, C266 to C271, C267 to C272, R107 to R110, R108 to R111, R109 to R112, R110 to R113, R111 to R114, R112 to R115, R113 to R116, U14 to U19
