File: hardware/FT2232HL.kicad_sch (KiCad schematic)
At the start: 46 parts, among them IC6 FT2232HL-TRAY, IC7 AT93C46DN-SH-B, P1 USB_C_Plug_USB2.0, U11 LM2937IMP-3.3, Y1 12Mhz

Commit message: Update hardware design and include board logo
Sync the saved schematics, PCB, project settings, and referenced custom
libraries with the updated design. Include the LOGO footprint and register
it in the project footprint table. The board now contains 524 footprints.

Keep unused source libraries, autosaves, backups, analysis outputs, and
manufacturing files out of the import. Point BOM exports to the existing
ignored production directory instead of a workstation-specific location.

Validation with KiCad 9.0.1:
- Netlist export succeeds and referenced custom libraries resolve.
- DRC: 0 errors, 40 warnings, 0 unconnected items, 0 schematic mismatches.
- ERC: 27 errors and 71 warnings, identical to the source design.

The pre-existing missing JTAG 3D model (87831-1420.stp) is not supplied by
the source project and remains unresolved.
Parts:
- added C222: 0.1u, Capacitor_SMD:C_0603_1608Metric, symbol Device:C_Small
- added R91: 4.7k, Resistor_SMD:R_0603_1608Metric, symbol Device:R
- added R92: 10k, Resistor_SMD:R_0603_1608Metric, symbol Device:R
- added U13: TPD2EUSB30, Package_TO_SOT_SMD:Texas_DRT-3, symbol Power_Protection:TPD2EUSB30
- C202: renamed from C198; value 1u -> 0.1u; LCSC C90057 -> C77055
- C203: renamed from C199; value 1u -> 47u; footprint Capacitor_SMD:C_0603_1608Metric -> Capacitor_SMD:C_0805_2012Metric; LCSC C90057 -> C76636
- C220: renamed from C216; LCSC C162215 -> C107045
- C221: renamed from C217; LCSC C162215 -> C107045
- U12: renamed from U11; LCSC C2870902 -> C140265
- Y1: value 12Mhz -> 12MHz
- renumbered C200 to C204, C201 to C205, C202 to C206, C203 to C207, C204 to C208, C205 to C209, C206 to C210, C207 to C211, C208 to C212, C209 to C213, C210 to C214, C211 to C215, C212 to C216, C213 to C217, C214 to C218, C215 to C219, R82 to R83, R83 to R84, R84 to R85, R85 to R86, R86 to R87, R87 to R88, R88 to R89, R89 to R90
Connections:
- net BCBUS7: now also R91.2, R92.1; no longer RN12.5
- net D+: now also U13.1 (D+)
- net D-: now also U13.2 (D-)
- net GND: now also C222.2, R92.2, U13.3 (GND)
- net VBUS_FT323H: now also C222.1, R91.1
- no-connect marks 1 -> 3
Other:
- moved on the sheet: FL1
