File: hardware/FT600Q.kicad_sch (KiCad schematic)
At the start: 37 parts, among them J8 692221030100, U12 LM2937IMP-3.3, U13 FT600, Y2 30Mhz

Commit message: Update hardware design and include board logo
Sync the saved schematics, PCB, project settings, and referenced custom
libraries with the updated design. Include the LOGO footprint and register
it in the project footprint table. The board now contains 524 footprints.

Keep unused source libraries, autosaves, backups, analysis outputs, and
manufacturing files out of the import. Point BOM exports to the existing
ignored production directory instead of a workstation-specific location.

Validation with KiCad 9.0.1:
- Netlist export succeeds and referenced custom libraries resolve.
- DRC: 0 errors, 40 warnings, 0 unconnected items, 0 schematic mismatches.
- ERC: 27 errors and 71 warnings, identical to the source design.

The pre-existing missing JTAG 3D model (87831-1420.stp) is not supplied by
the source project and remains unresolved.
Parts:
- added U15, U17, U18: TPD2EUSB30, Package_TO_SOT_SMD:Texas_DRT-3, symbol Power_Protection:TPD2EUSB30
- C228: renamed from C223; value 1u -> 0.1u; LCSC C90057 -> C77055
- C229: renamed from C224; value 1u -> 10u; footprint Capacitor_SMD:C_0603_1608Metric -> Capacitor_SMD:C_0805_2012Metric; LCSC C90057 -> C440198
- C238: renamed from C233; LCSC C90057 -> C90057
- FL2, FL3, FL4: LCSC DLM0NSN500HY2D -> C1857796
- U14: renamed from U12; LCSC C2870902 -> C140265
- Y2: value 30Mhz -> 30MHz; LCSC C112563 -> C19272757
- renumbered C218 to C223, C219 to C224, C220 to C225, C221 to C226, C222 to C227, C225 to C230, C226 to C231, C227 to C232, C228 to C233, C229 to C234, C230 to C235, C231 to C236, C232 to C237, C234 to C239, C235 to C240, C236 to C241, C237 to C242, C238 to C243, C239 to C244, R90 to R93, R91 to R94, R92 to R95, U13 to U16
Connections:
- net FT600_D+: now also U15.1 (D+)
- net FT600_D-: now also U15.2 (D-)
- net GND: now also U15.3 (GND), U17.3 (GND), U18.3 (GND); no longer U16.14 (GND)
- net SSRX+: now also U18.1 (D+)
- net SSRX-: now also U18.2 (D-)
- net SSTX+: now also U17.1 (D+)
- net SSTX-: now also U17.2 (D-)
- no-connect marks 0 -> 1
Other:
- moved on the sheet: FB11, FB12, FB13, J8
