File: hardware/MainFPGAConfig.kicad_sch (KiCad schematic)
At the start: 29 parts, among them J4 JTAG_CONFIG, SW1 SW_DIP_x03, U3 XC7S100-2FGGA484I, U5 IS25LP064A-JLLE, U6 SN74LVC2G17DCKRE4, U7 SN74LVC2G17DCKRE4

Commit message: Update hardware design and include board logo
Sync the saved schematics, PCB, project settings, and referenced custom
libraries with the updated design. Include the LOGO footprint and register
it in the project footprint table. The board now contains 524 footprints.

Keep unused source libraries, autosaves, backups, analysis outputs, and
manufacturing files out of the import. Point BOM exports to the existing
ignored production directory instead of a workstation-specific location.

Validation with KiCad 9.0.1:
- Netlist export succeeds and referenced custom libraries resolve.
- DRC: 0 errors, 40 warnings, 0 unconnected items, 0 schematic mismatches.
- ERC: 27 errors and 71 warnings, identical to the source design.

The pre-existing missing JTAG 3D model (87831-1420.stp) is not supplied by
the source project and remains unresolved.
Parts:
- D2: value G_LED -> B_LED; LCSC C5342733 -> C19171394
- R34: renamed from R33; LCSC C99782 -> C22548
- R35: renamed from R34; LCSC C99782 -> C22548
- R36: renamed from R35; LCSC C99782 -> C22548
- renumbered C186 to C190, C187 to C191, C188 to C192, R30 to R31, R31 to R32, R32 to R33, R36 to R37, R37 to R38, R38 to R39, R39 to R40, R40 to R41, R41 to R42, R42 to R43, R43 to R44, R44 to R45, R45 to R46, R46 to R47, U3 to U4, U5 to U6, U6 to U7, U7 to U8
