File: hardware/MainFPGAHeader.kicad_sch (KiCad schematic)
At the start: 4 parts, among them J6 PIN_Socket_2x20

Commit message: Update hardware design and include board logo
Sync the saved schematics, PCB, project settings, and referenced custom
libraries with the updated design. Include the LOGO footprint and register
it in the project footprint table. The board now contains 524 footprints.

Keep unused source libraries, autosaves, backups, analysis outputs, and
manufacturing files out of the import. Point BOM exports to the existing
ignored production directory instead of a workstation-specific location.

Validation with KiCad 9.0.1:
- Netlist export succeeds and referenced custom libraries resolve.
- DRC: 0 errors, 40 warnings, 0 unconnected items, 0 schematic mismatches.
- ERC: 27 errors and 71 warnings, identical to the source design.

The pre-existing missing JTAG 3D model (87831-1420.stp) is not supplied by
the source project and remains unresolved.
Parts:
- C196: renamed from C192; footprint Capacitor_SMD:C_0603_1608Metric -> Capacitor_SMD:C_0805_2012Metric; LCSC C77386 -> C126592
- renumbered C193 to C197, C194 to C198
Changed lines of the file:
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@@
 		(dnp no)
 		(fields_autoplaced yes)
-		(property "Reference" "C194"
+		(property "Reference" "C198"
 			(at 172.72 71.1199 0)
 			(effects
@@
 			(project "shamiko"
 				(path "/3bdb682e-16f1-4662-9b00-b0c9070eb240/3ffd7f99-7fa4-43ca-b8b7-24af26783d6d"
-					(reference "C194")
+					(reference "C198")
 					(unit 1)
 				)
@@
 		(dnp no)
 		(fields_autoplaced yes)
-		(property "Reference" "#PWR0248"
+		(property "Reference" "#PWR0247"
 			(at 73.66 34.29 0)
 			(effects
@@
 			(project ""
 				(path "/3bdb682e-16f1-4662-9b00-b0c9070eb240/3ffd7f99-7fa4-43ca-b8b7-24af26783d6d"
-					(reference "#PWR0248")
+					(reference "#PWR0247")
 					(unit 1)
 				)
@@
 		(dnp no)
 		(fields_autoplaced yes)
-		(property "Reference" "#PWR0253"
+		(property "Reference" "#PWR0252"
 			(at 168.91 100.33 0)
 			(effects
@@
 			(project "shamiko"
 				(path "/3bdb682e-16f1-4662-9b00-b0c9070eb240/3ffd7f99-7fa4-43ca-b8b7-24af26783d6d"
-					(reference "#PWR0253")
+					(reference "#PWR0252")
 					(unit 1)
 				)
@@
 		(dnp no)
 		(fields_autoplaced yes)
-		(property "Reference" "#PWR0250"
+		(property "Reference" "#PWR0249"
 			(at 156.21 54.61 0)
 			(effects
@@
 			(project "shamiko"
 				(path "/3bdb682e-16f1-4662-9b00-b0c9070eb240/3ffd7f99-7fa4-43ca-b8b7-24af26783d6d"
-					(reference "#PWR0250")
+					(reference "#PWR0249")
 					(unit 1)
 				)
@@
 		(dnp no)
 		(fields_autoplaced yes)
-		(property "Reference" "#PWR0247"
+		(property "Reference" "#PWR0246"
 			(at 67.31 34.29 0)
 			(effects
@@
 			(project "shamiko"
 				(path "/3bdb682e-16f1-4662-9b00-b0c9070eb240/3ffd7f99-7fa4-43ca-b8b7-24af26783d6d"
-					(reference "#PWR0247")
+					(reference "#PWR0246")
 					(unit 1)
 				)
@@
 		(dnp no)
 		(fields_autoplaced yes)
-		(property "Reference" "#PWR0254"
+		(property "Reference" "#PWR0253"
 			(at 86.36 147.32 0)
 			(effects
@@
 			(project ""
 				(path "/3bdb682e-16f1-4662-9b00-b0c9070eb240/3ffd7f99-7fa4-43ca-b8b7-24af26783d6d"
-					(reference "#PWR0254")
+					(reference "#PWR0253")
 					(unit 1)
 				)
@@
 		(dnp no)
 		(fields_autoplaced yes)
-		(property "Reference" "#PWR0251"
+		(property "Reference" "#PWR0250"
 			(at 143.51 100.33 0)
 			(effects
@@
 			(project "shamiko"
 				(path "/3bdb682e-16f1-4662-9b00-b0c9070eb240/3ffd7f99-7fa4-43ca-b8b7-24af26783d6d"
-					(reference "#PWR0251")
+					(reference "#PWR0250")
 					(unit 1)
 				)
@@
 		(dnp no)
 		(fields_autoplaced yes)
-		(property "Reference" "C192"
+		(property "Reference" "C196"
 			(at 147.32 71.1199 0)
 			(effects
@@
 			)
 		)
-		(property "Footprint" "Capacitor_SMD:C_0603_1608Metric"
+		(property "Footprint" "Capacitor_SMD:C_0805_2012Metric"
 			(at 144.4752 76.2 0)
 			(effects
@@
 			)
 		)
-		(property "LCSC" "C77386 "
+		(property "LCSC" "C126592"
 			(at 143.51 72.39 0)
 			(effects
@@
 			(project ""
 				(path "/3bdb682e-16f1-4662-9b00-b0c9070eb240/3ffd7f99-7fa4-43ca-b8b7-24af26783d6d"
-					(reference "C192")
+					(reference "C196")
 					(unit 1)
 				)
@@
 		(dnp no)
 		(fields_autoplaced yes)
-		(property "Reference" "#PWR0249"
+		(property "Reference" "#PWR0248"
 			(at 143.51 54.61 0)
 			(effects
@@
 			(project "shamiko"
 				(path "/3bdb682e-16f1-4662-9b00-b0c9070eb240/3ffd7f99-7fa4-43ca-b8b7-24af26783d6d"
-					(reference "#PWR0249")
+					(reference "#PWR0248")
 					(unit 1)
 				)
@@
 		(dnp no)
 		(fields_autoplaced yes)
-		(property "Reference" "#PWR0252"
+		(property "Reference" "#PWR0251"
 			(at 156.21 100.33 0)
 			(effects
@@
 			(project "shamiko"
 				(path "/3bdb682e-16f1-4662-9b00-b0c9070eb240/3ffd7f99-7fa4-43ca-b8b7-24af26783d6d"
-					(reference "#PWR0252")
+					(reference "#PWR0251")
 					(unit 1)
 				)
@@
 		(dnp no)
 		(fields_autoplaced yes)
-		(property "Reference" "C193"
+		(property "Reference" "C197"
 			(at 160.02 71.1199 0)
 			(effects
@@
 			(project "shamiko"
 				(path "/3bdb682e-16f1-4662-9b00-b0c9070eb240/3ffd7f99-7fa4-43ca-b8b7-24af26783d6d"
-					(reference "C193")
-					(unit 1)
-				)
+					(reference "C197")
+					(unit 1)
+				)
