File: hardware/MainFPGAIO.kicad_sch (KiCad schematic)
At the start: 1 part, among them U3 XC7S100-2FGGA484I

Commit message: Update hardware design and include board logo
Sync the saved schematics, PCB, project settings, and referenced custom
libraries with the updated design. Include the LOGO footprint and register
it in the project footprint table. The board now contains 524 footprints.

Keep unused source libraries, autosaves, backups, analysis outputs, and
manufacturing files out of the import. Point BOM exports to the existing
ignored production directory instead of a workstation-specific location.

Validation with KiCad 9.0.1:
- Netlist export succeeds and referenced custom libraries resolve.
- DRC: 0 errors, 40 warnings, 0 unconnected items, 0 schematic mismatches.
- ERC: 27 errors and 71 warnings, identical to the source design.

The pre-existing missing JTAG 3D model (87831-1420.stp) is not supplied by
the source project and remains unresolved.
Parts:
- renumbered U3 to U4
Changed lines of the file:
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@@
 		(on_board yes)
 		(dnp no)
-		(property "Reference" "U3"
+		(property "Reference" "U4"
 			(at 64.135 158.75 0)
 			(effects
@@
 			(project "shamiko"
 				(path "/3bdb682e-16f1-4662-9b00-b0c9070eb240/05e58379-3136-4784-a311-aa48fe232d95"
-					(reference "U3")
+					(reference "U4")
 					(unit 9)
 				)
@@
 		(on_board yes)
 		(dnp no)
-		(property "Reference" "U3"
+		(property "Reference" "U4"
 			(at 217.805 13.97 0)
 			(effects
@@
 			(project "shamiko"
 				(path "/3bdb682e-16f1-4662-9b00-b0c9070eb240/05e58379-3136-4784-a311-aa48fe232d95"
-					(reference "U3")
+					(reference "U4")
 					(unit 13)
 				)
@@
 		(on_board yes)
 		(dnp no)
-		(property "Reference" "U3"
+		(property "Reference" "U4"
 			(at 133.985 148.59 0)
 			(effects
@@
 			(project ""
 				(path "/3bdb682e-16f1-4662-9b00-b0c9070eb240/05e58379-3136-4784-a311-aa48fe232d95"
-					(reference "U3")
+					(reference "U4")
 					(unit 12)
 				)
@@
 		(on_board yes)
 		(dnp no)
-		(property "Reference" "U3"
+		(property "Reference" "U4"
 			(at 133.985 12.7 0)
 			(effects
@@
 			(project ""
 				(path "/3bdb682e-16f1-4662-9b00-b0c9070eb240/05e58379-3136-4784-a311-aa48fe232d95"
-					(reference "U3")
+					(reference "U4")
 					(unit 14)
 				)
@@
 		(on_board yes)
 		(dnp no)
-		(property "Reference" "U3"
+		(property "Reference" "U4"
 			(at 374.015 13.97 0)
 			(effects
@@
 			(project "shamiko"
 				(path "/3bdb682e-16f1-4662-9b00-b0c9070eb240/05e58379-3136-4784-a311-aa48fe232d95"
-					(reference "U3")
+					(reference "U4")
 					(unit 10)
 				)
@@
 		(on_board yes)
 		(dnp no)
-		(property "Reference" "U3"
+		(property "Reference" "U4"
 			(at 64.135 13.97 0)
 			(effects
@@
 			(project ""
 				(path "/3bdb682e-16f1-4662-9b00-b0c9070eb240/05e58379-3136-4784-a311-aa48fe232d95"
-					(reference "U3")
+					(reference "U4")
 					(unit 15)
 				)
@@
 		(on_board yes)
 		(dnp no)
-		(property "Reference" "U3"
+		(property "Reference" "U4"
 			(at 299.085 13.97 0)
 			(effects
@@
 			(project ""
 				(path "/3bdb682e-16f1-4662-9b00-b0c9070eb240/05e58379-3136-4784-a311-aa48fe232d95"
-					(reference "U3")
+					(reference "U4")
 					(unit 11)
 				)
