File: hardware/MainFPGAPeripheral.kicad_sch (KiCad schematic)
At the start: 24 parts, among them SW3 SW_MEC_5E, SW4 SW_MEC_5E, SW5 SW_MEC_5E, SW6 SW_MEC_5E, SW7 SW_DIP_x08

Commit message: Update hardware design and include board logo
Sync the saved schematics, PCB, project settings, and referenced custom
libraries with the updated design. Include the LOGO footprint and register
it in the project footprint table. The board now contains 524 footprints.

Keep unused source libraries, autosaves, backups, analysis outputs, and
manufacturing files out of the import. Point BOM exports to the existing
ignored production directory instead of a workstation-specific location.

Validation with KiCad 9.0.1:
- Netlist export succeeds and referenced custom libraries resolve.
- DRC: 0 errors, 40 warnings, 0 unconnected items, 0 schematic mismatches.
- ERC: 27 errors and 71 warnings, identical to the source design.

The pre-existing missing JTAG 3D model (87831-1420.stp) is not supplied by
the source project and remains unresolved.
Parts:
- renumbered R64 to R65, R65 to R66, R66 to R67, R67 to R68, R68 to R69, R69 to R70, R70 to R71, R71 to R72
Changed lines of the file:
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@@
 		(dnp no)
 		(fields_autoplaced yes)
-		(property "Reference" "R67"
+		(property "Reference" "R68"
 			(at 220.98 36.8299 0)
 			(effects
@@
 			(project "shamiko"
 				(path "/3bdb682e-16f1-4662-9b00-b0c9070eb240/d82c4c14-c0a7-4141-a905-05355b270ee6"
-					(reference "R67")
+					(reference "R68")
 					(unit 1)
 				)
@@
 		(dnp no)
 		(fields_autoplaced yes)
-		(property "Reference" "#PWR0264"
+		(property "Reference" "#PWR0263"
 			(at 77.47 129.54 0)
 			(effects
@@
 			(project ""
 				(path "/3bdb682e-16f1-4662-9b00-b0c9070eb240/d82c4c14-c0a7-4141-a905-05355b270ee6"
-					(reference "#PWR0264")
+					(reference "#PWR0263")
 					(unit 1)
 				)
@@
 		(dnp no)
 		(fields_autoplaced yes)
-		(property "Reference" "R68"
+		(property "Reference" "R69"
 			(at 233.68 36.8299 0)
 			(effects
@@
 			(project "shamiko"
 				(path "/3bdb682e-16f1-4662-9b00-b0c9070eb240/d82c4c14-c0a7-4141-a905-05355b270ee6"
-					(reference "R68")
+					(reference "R69")
 					(unit 1)
 				)
@@
 		(dnp no)
 		(fields_autoplaced yes)
-		(property "Reference" "R71"
+		(property "Reference" "R72"
 			(at 271.78 36.8299 0)
 			(effects
@@
 			(project "shamiko"
 				(path "/3bdb682e-16f1-4662-9b00-b0c9070eb240/d82c4c14-c0a7-4141-a905-05355b270ee6"
-					(reference "R71")
+					(reference "R72")
 					(unit 1)
 				)
@@
 		(dnp no)
 		(fields_autoplaced yes)
-		(property "Reference" "R69"
+		(property "Reference" "R70"
 			(at 246.38 36.8299 0)
 			(effects
@@
 			(project "shamiko"
 				(path "/3bdb682e-16f1-4662-9b00-b0c9070eb240/d82c4c14-c0a7-4141-a905-05355b270ee6"
-					(reference "R69")
+					(reference "R70")
 					(unit 1)
 				)
@@
 		(dnp no)
 		(fields_autoplaced yes)
-		(property "Reference" "R65"
+		(property "Reference" "R66"
 			(at 195.58 36.8299 0)
 			(effects
@@
 			(project ""
 				(path "/3bdb682e-16f1-4662-9b00-b0c9070eb240/d82c4c14-c0a7-4141-a905-05355b270ee6"
-					(reference "R65")
+					(reference "R66")
 					(unit 1)
 				)
@@
 		(dnp no)
 		(fields_autoplaced yes)
-		(property "Reference" "R66"
+		(property "Reference" "R67"
 			(at 208.28 36.8299 0)
 			(effects
@@
 			(project "shamiko"
 				(path "/3bdb682e-16f1-4662-9b00-b0c9070eb240/d82c4c14-c0a7-4141-a905-05355b270ee6"
-					(reference "R66")
+					(reference "R67")
 					(unit 1)
 				)
@@
 		(dnp no)
 		(fields_autoplaced yes)
-		(property "Reference" "R64"
+		(property "Reference" "R65"
 			(at 182.88 36.8299 0)
 			(effects
@@
 			(project ""
 				(path "/3bdb682e-16f1-4662-9b00-b0c9070eb240/d82c4c14-c0a7-4141-a905-05355b270ee6"
-					(reference "R64")
+					(reference "R65")
 					(unit 1)
 				)
@@
 		(dnp no)
 		(fields_autoplaced yes)
-		(property "Reference" "R70"
+		(property "Reference" "R71"
 			(at 259.08 36.8299 0)
 			(effects
@@
 			(project "shamiko"
 				(path "/3bdb682e-16f1-4662-9b00-b0c9070eb240/d82c4c14-c0a7-4141-a905-05355b270ee6"
-					(reference "R70")
+					(reference "R71")
 					(unit 1)
 				)
@@
 		(dnp no)
 		(fields_autoplaced yes)
-		(property "Reference" "#PWR0263"
+		(property "Reference" "#PWR0262"
 			(at 49.53 129.54 0)
 			(effects
@@
 			(project "shamiko"
 				(path "/3bdb682e-16f1-4662-9b00-b0c9070eb240/d82c4c14-c0a7-4141-a905-05355b270ee6"
-					(reference "#PWR0263")
+					(reference "#PWR0262")
 					(unit 1)
 				)
