File: hardware/MainFPGAPower.kicad_sch (KiCad schematic)
At the start: 89 parts, among them U3 XC7S100-2FGGA484I

Commit message: Update hardware design and include board logo
Sync the saved schematics, PCB, project settings, and referenced custom
libraries with the updated design. Include the LOGO footprint and register
it in the project footprint table. The board now contains 524 footprints.

Keep unused source libraries, autosaves, backups, analysis outputs, and
manufacturing files out of the import. Point BOM exports to the existing
ignored production directory instead of a workstation-specific location.

Validation with KiCad 9.0.1:
- Netlist export succeeds and referenced custom libraries resolve.
- DRC: 0 errors, 40 warnings, 0 unconnected items, 0 schematic mismatches.
- ERC: 27 errors and 71 warnings, identical to the source design.

The pre-existing missing JTAG 3D model (87831-1420.stp) is not supplied by
the source project and remains unresolved.
Parts:
- C100: renamed from C96; LCSC C90057 -> C90057
- C103: renamed from C99; LCSC C90057 -> C90057
- C104: renamed from C100; LCSC C90057 -> C90057
- C113: renamed from C109; LCSC C90057 -> C90057
- C114: renamed from C110; LCSC C90057 -> C90057
- C117: renamed from C113; LCSC C90057 -> C90057
- C118: renamed from C114; LCSC C90057 -> C90057
- C119: renamed from C115; LCSC C90057 -> C90057
- C129: renamed from C125; LCSC C90057 -> C90057
- C132: renamed from C128; LCSC C85973 -> C15195
- C61: renamed from C57; LCSC C90057 -> C90057
- C62: renamed from C58; LCSC C90057 -> C90057
- C71: renamed from C67; LCSC C90057 -> C90057
- C72: renamed from C68; LCSC C90057 -> C90057
- C75: renamed from C71; LCSC C90057 -> C90057
- C76: renamed from C72; LCSC C90057 -> C90057
- C85: renamed from C81; LCSC C90057 -> C90057
- C86: renamed from C82; LCSC C90057 -> C90057
- C89: renamed from C85; LCSC C90057 -> C90057
- C90: renamed from C86; LCSC C90057 -> C90057
- C99: renamed from C95; LCSC C90057 -> C90057
- renumbered C97 to C101, C98 to C102, C101 to C105, C102 to C106, C103 to C107, C104 to C108, C105 to C109, C106 to C110, C107 to C111, C108 to C112, C111 to C115, C112 to C116, C116 to C120, C117 to C121, C118 to C122, C119 to C123, C120 to C124, C121 to C125, C122 to C126, C123 to C127, C124 to C128, C126 to C130, C127 to C131, C129 to C133, C130 to C134, C131 to C135, C132 to C136, C133 to C137, C134 to C138, C135 to C139, C136 to C140, C137 to C141, C138 to C142, C139 to C143, C140 to C144, C141 to C145, C56 to C60, C59 to C63, C60 to C64, C61 to C65, C62 to C66, C63 to C67, C64 to C68, C65 to C69, C66 to C70, C69 to C73, C70 to C74, C73 to C77, C74 to C78, C75 to C79, C76 to C80, C77 to C81, C78 to C82, C79 to C83, C80 to C84, C83 to C87, C84 to C88, C87 to C91, C88 to C92, C89 to C93, C90 to C94, C91 to C95, C92 to C96, C93 to C97, C94 to C98, U3 to U4
