File: hardware/MainFPGASupervisor.kicad_sch (KiCad schematic)
At the start: 22 parts, among them J10 SMA, J9 SMA, SW11 SW_MEC_5E, SW12 SW_MEC_5E, Y3 HCI 1532P-48.000KWVDT

Commit message: Update hardware design and include board logo
Sync the saved schematics, PCB, project settings, and referenced custom
libraries with the updated design. Include the LOGO footprint and register
it in the project footprint table. The board now contains 524 footprints.

Keep unused source libraries, autosaves, backups, analysis outputs, and
manufacturing files out of the import. Point BOM exports to the existing
ignored production directory instead of a workstation-specific location.

Validation with KiCad 9.0.1:
- Netlist export succeeds and referenced custom libraries resolve.
- DRC: 0 errors, 40 warnings, 0 unconnected items, 0 schematic mismatches.
- ERC: 27 errors and 71 warnings, identical to the source design.

The pre-existing missing JTAG 3D model (87831-1420.stp) is not supplied by
the source project and remains unresolved.
Parts:
- C250: renamed from C245; now not fitted
- R100: renamed from R97; LCSC C95204 -> C2906993
- R101: renamed from R98; LCSC C95204 -> C862232
- R102: renamed from R99; LCSC C95204 -> C105579
- Y3: value HCI 1532P-48.000KWVDT -> HCI 1532H-48.000GWVATS
- renumbered C240 to C245, C241 to C246, C242 to C247, C243 to C248, C244 to C249, C246 to C251, R93 to R96, R94 to R97, R95 to R98, R96 to R99
Changed lines of the file:
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@@
 		(on_board yes)
 		(dnp no)
-		(property "Reference" "C243"
+		(property "Reference" "C248"
 			(at 101.6 40.386 0)
 			(effects
@@
 			(project "shamiko"
 				(path "/3bdb682e-16f1-4662-9b00-b0c9070eb240/5331855a-6100-4742-b2a4-dc6f2f418ddc"
-					(reference "C243")
+					(reference "C248")
 					(unit 1)
 				)
@@
 		(on_board yes)
 		(dnp no)
-		(property "Reference" "#PWR0340"
+		(property "Reference" "#PWR0345"
 			(at 189.23 152.4 0)
 			(effects
@@
 			(project "shamiko"
 				(path "/3bdb682e-16f1-4662-9b00-b0c9070eb240/5331855a-6100-4742-b2a4-dc6f2f418ddc"
-					(reference "#PWR0340")
+					(reference "#PWR0345")
 					(unit 1)
 				)
@@
 			)
 		)
-		(property "Value" "HCI 1532P-48.000KWVDT"
+		(property "Value" "HCI 1532H-48.000GWVATS"
 			(at 77.216 54.864 0)
 			(effects
@@
 		(on_board yes)
 		(dnp no)
-		(property "Reference" "#PWR0333"
+		(property "Reference" "#PWR0338"
 			(at 101.6 52.07 0)
 			(effects
@@
 			(project "shamiko"
 				(path "/3bdb682e-16f1-4662-9b00-b0c9070eb240/5331855a-6100-4742-b2a4-dc6f2f418ddc"
-					(reference "#PWR0333")
+					(reference "#PWR0338")
 					(unit 1)
 				)
@@
 		(on_board yes)
 		(dnp no)
-		(property "Reference" "#PWR0339"
+		(property "Reference" "#PWR0344"
 			(at 179.07 152.4 0)
 			(effects
@@
 			(project "shamiko"
 				(path "/3bdb682e-16f1-4662-9b00-b0c9070eb240/5331855a-6100-4742-b2a4-dc6f2f418ddc"
-					(reference "#PWR0339")
+					(reference "#PWR0344")
 					(unit 1)
 				)
@@
 		(on_board yes)
 		(dnp no)
-		(property "Reference" "#PWR0336"
+		(property "Reference" "#PWR0341"
 			(at 105.41 85.09 0)
 			(effects
@@
 			(project "shamiko"
 				(path "/3bdb682e-16f1-4662-9b00-b0c9070eb240/5331855a-6100-4742-b2a4-dc6f2f418ddc"
-					(reference "#PWR0336")
+					(reference "#PWR0341")
 					(unit 1)
 				)
@@
 		(on_board yes)
 		(dnp no)
-		(property "Reference" "R94"
+		(property "Reference" "R97"
 			(at 123.19 55.626 90)
 			(effects
@@
 			(project ""
 				(path "/3bdb682e-16f1-4662-9b00-b0c9070eb240/5331855a-6100-4742-b2a4-dc6f2f418ddc"
-					(reference "R94")
+					(reference "R97")
 					(unit 1)
 				)
@@
 		(on_board yes)
 		(dnp no)
-		(property "Reference" "R95"
+		(property "Reference" "R98"
 			(at 30.226 68.58 90)
 			(effects
@@
 			(project "shamiko"
 				(path "/3bdb682e-16f1-4662-9b00-b0c9070eb240/5331855a-6100-4742-b2a4-dc6f2f418ddc"
-					(reference "R95")
+					(reference "R98")
 					(unit 1)
 				)
@@
 		(on_board yes)
 		(dnp no)
-		(property "Reference" "#PWR0332"
+		(property "Reference" "#PWR0337"
 			(at 90.17 52.07 0)
 			(effects
@@
 			(project "shamiko"
 				(path "/3bdb682e-16f1-4662-9b00-b0c9070eb240/5331855a-6100-4742-b2a4-dc6f2f418ddc"
-					(reference "#PWR0332")
+					(reference "#PWR0337")
 					(unit 1)
 				)
@@
 		(dnp no)
 		(fields_autoplaced yes)
-		(property "Reference" "#PWR0338"
+		(property "Reference" "#PWR0343"
 			(at 48.26 121.92 0)
 			(effects
@@
 			(project ""
 				(path "/3bdb682e-16f1-4662-9b00-b0c9070eb240/5331855a-6100-4742-b2a4-dc6f2f418ddc"
-					(reference "#PWR0338")
+					(reference "#PWR0343")
 					(unit 1)
 				)
@@
 		(on_board yes)
 		(dnp no)
-		(property "Reference" "R99"
+		(property "Reference" "R102"
 			(at 269.494 112.014 0)
 			(effects
@@
 			)
 		)
-		(property "LCSC" "C95204"
+		(property "LCSC" "C105579"
 			(at 265.43 114.3 0)
 			(effects
@@
 			(project "shamiko"
 				(path "/3bdb682e-16f1-4662-9b00-b0c9070eb240/5331855a-6100-4742-b2a4-dc6f2f418ddc"
-					(reference "R99")
+					(reference "R102")
 					(unit 1)
 				)
@@
 		(on_board yes)
 		(dnp no)
-		(property "Reference" "#PWR0341"
+		(property "Reference" "#PWR0346"
 			(at 198.12 152.4 0)
 			(effects
@@
 			(project "shamiko"
 				(path "/3bdb682e-16f1-4662-9b00-b0c9070eb240/5331855a-6100-4742-b2a4-dc6f2f418ddc"
-					(reference "#PWR0341")
+					(reference "#PWR0346")
 					(unit 1)
 				)
@@
 		(on_board yes)
 		(dnp no)
-		(property "Reference" "#PWR0342"
+		(property "Reference" "#PWR0347"
 			(at 234.95 152.4 0)
 			(effects
@@
 			(project "shamiko"
 				(path "/3bdb682e-16f1-4662-9b00-b0c9070eb240/5331855a-6100-4742-b2a4-dc6f2f418ddc"
-					(reference "#PWR0342")
+					(reference "#PWR0347")
 					(unit 1)
 				)
@@
 		(on_board yes)
 		(dnp no)
-		(property "Reference" "#PWR0343"
+		(property "Reference" "#PWR0348"
 			(at 248.92 152.4 0)
 			(effects
@@
 			(project "shamiko"
 				(path "/3bdb682e-16f1-4662-9b00-b0c9070eb240/5331855a-6100-4742-b2a4-dc6f2f418ddc"
-					(reference "#PWR0343")
+					(reference "#PWR0348")
 					(unit 1)
 				)
@@
 		(on_board yes)
 		(dnp no)
-		(property "Reference" "#PWR0335"
+		(property "Reference" "#PWR0340"
 			(at 215.9 69.85 0)
 			(effects
@@
 			(project "shamiko"
 				(path "/3bdb682e-16f1-4662-9b00-b0c9070eb240/5331855a-6100-4742-b2a4-dc6f2f418ddc"
-					(reference "#PWR0335")
+					(reference "#PWR0340")
 					(unit 1)
 				)
@@
 		(on_board yes)
 		(dnp no)
-		(property "Reference" "C246"
+		(property "Reference" "C251"
 			(at 248.92 121.666 0)
 			(effects
@@
 			(project "shamiko"
 				(path "/3bdb682e-16f1-4662-9b00-b0c9070eb240/5331855a-6100-4742-b2a4-dc6f2f418ddc"
-					(reference "C246")
+					(reference "C251")
 					(unit 1)
 				)
@@
 		(on_board yes)
 		(dnp no)
-		(property "Reference" "C240"
+		(property "Reference" "C245"
 			(at 94.742 39.116 0)
 			(effects
@@
 			(project "shamiko"
 				(path "/3bdb682e-16f1-4662-9b00-b0c9070eb240/5331855a-6100-4742-b2a4-dc6f2f418ddc"
-					(reference "C240")
+					(reference "C245")
 					(unit 1)
 				)
@@
 		(on_board yes)
 		(dnp no)
-		(property "Reference" "R93"
+		(property "Reference" "R96"
 			(at 40.386 50.8 90)
 			(effects
@@
 			(project "shamiko"
 				(path "/3bdb682e-16f1-4662-9b00-b0c9070eb240/5331855a-6100-4742-b2a4-dc6f2f418ddc"
-					(reference "R93")
+					(reference "R96")
 					(unit 1)
 				)
@@
 		(on_board yes)
 		(dnp no)
-		(property "Reference" "R97"
+		(property "Reference" "R100"
 			(at 269.494 97.028 0)
 			(effects
@@
 			)
 		)
-		(property "LCSC" "C95204"
+		(property "LCSC" "C2906993"
 			(at 265.43 99.06 0)
 			(effects
@@
 			(project "shamiko"
 				(path "/3bdb682e-16f1-4662-9b00-b0c9070eb240/5331855a-6100-4742-b2a4-dc6f2f418ddc"
-					(reference "R97")
+					(reference "R100")
 					(unit 1)
 				)
@@
 		(on_board yes)
 		(dnp no)
-		(property "Reference" "#PWR0344"
+		(property "Reference" "#PWR0349"
 			(at 265.43 153.67 0)
 			(effects
@@
 			(project "shamiko"
 				(path "/3bdb682e-16f1-4662-9b00-b0c9070eb240/5331855a-6100-4742-b2a4-dc6f2f418ddc"
-					(reference "#PWR0344")
+					(reference "#PWR0349")
 					(unit 1)
 				)
@@
 		(on_board yes)
 		(dnp no)
-		(property "Reference" "C241"
+		(property "Reference" "C246"
 			(at 215.9 39.116 0)
 			(effects
@@
 			(project "shamiko"
 				(path "/3bdb682e-16f1-4662-9b00-b0c9070eb240/5331855a-6100-4742-b2a4-dc6f2f418ddc"
-					(reference "C241")
+					(reference "C246")
 					(unit 1)
 				)
@@
 		(on_board yes)
 		(dnp no)
-		(property "Reference" "#PWR0334"
+		(property "Reference" "#PWR0339"
 			(at 187.96 69.85 0)
 			(effects
@@
 			(project "shamiko"
 				(path "/3bdb682e-16f1-4662-9b00-b0c9070eb240/5331855a-6100-4742-b2a4-dc6f2f418ddc"
-					(reference "#PWR0334")
+					(reference "#PWR0339")
 					(unit 1)
 				)
@@
 		(on_board yes)
 		(dnp no)
-		(property "Reference" "C242"
+		(property "Reference" "C247"
 			(at 78.74 40.386 0)
 			(effects
@@
 			(project "shamiko"
 				(path "/3bdb682e-16f1-4662-9b00-b0c9070eb240/5331855a-6100-4742-b2a4-dc6f2f418ddc"
-					(reference "C242")
+					(reference "C247")
 					(unit 1)
 				)
@@
 		(on_board yes)
 		(dnp no)
-		(property "Reference" "#PWR0337"
+		(property "Reference" "#PWR0342"
 			(at 33.02 96.52 0)
 			(effects
@@
 			(project "shamiko"
 				(path "/3bdb682e-16f1-4662-9b00-b0c9070eb240/5331855a-6100-4742-b2a4-dc6f2f418ddc"
-					(reference "#PWR0337")
+					(reference "#PWR0342")
 					(unit 1)
 				)
@@
 		(on_board yes)
 		(dnp no)
-		(property "Reference" "C244"
+		(property "Reference" "C249"
 			(at 198.12 121.666 0)
 			(effects
@@
 			(project "shamiko"
 				(path "/3bdb682e-16f1-4662-9b00-b0c9070eb240/5331855a-6100-4742-b2a4-dc6f2f418ddc"
-					(reference "C244")
+					(reference "C249")
 					(unit 1)
 				)
@@
 		(in_bom yes)
 		(on_board yes)
-		(dnp no)
-		(property "Reference" "C245"
+		(dnp yes)
+		(property "Reference" "C250"
 			(at 234.95 121.666 0)
 			(effects
@@
 					(size 1.27 1.27)
 				)
+				(hide yes)
 			)
 		)
@@
 			(project "shamiko"
 				(path "/3bdb682e-16f1-4662-9b00-b0c9070eb240/5331855a-6100-4742-b2a4-dc6f2f418ddc"
-					(reference "C245")
+					(reference "C250")
 					(unit 1)
 				)
@@
 		(on_board yes)
 		(dnp no)
-		(property "Reference" "R98"
+		(property "Reference" "R101"
 			(at 171.45 111.506 90)
 			(effects
@@
 			)
 		)
-		(property "LCSC" "C95204"
+		(property "LCSC" "C862232"
 			(at 171.45 109.22 0)
 			(effects
@@
 			(project "shamiko"
 				(path "/3bdb682e-16f1-4662-9b00-b0c9070eb240/5331855a-6100-4742-b2a4-dc6f2f418ddc"
-					(reference "R98")
+					(reference "R101")
 					(unit 1)
 				)
@@
 		(on_board yes)
 		(dnp no)
-		(property "Reference" "#PWR0331"
+		(property "Reference" "#PWR0336"
 			(at 78.74 52.07 0)
 			(effects
@@
 			(project "shamiko"
 				(path "/3bdb682e-16f1-4662-9b00-b0c9070eb240/5331855a-6100-4742-b2a4-dc6f2f418ddc"
-					(reference "#PWR0331")
+					(reference "#PWR0336")
 					(unit 1)
 				)
@@
 		(dnp no)
 		(fields_autoplaced yes)
-		(property "Reference" "R96"
+		(property "Reference" "R99"
 			(at 191.77 93.9799 0)
 			(effects
@@
 			(project ""
 				(path "/3bdb682e-16f1-4662-9b00-b0c9070eb240/5331855a-6100-4742-b2a4-dc6f2f418ddc"
-					(reference "R96")
+					(reference "R99")
 					(unit 1)
 				)
