File: hardware/Power(VCC1V0C).kicad_sch (KiCad schematic)
At the start: 17 parts, among them IC2 LT3071

Commit message: Update hardware design and include board logo
Sync the saved schematics, PCB, project settings, and referenced custom
libraries with the updated design. Include the LOGO footprint and register
it in the project footprint table. The board now contains 524 footprints.

Keep unused source libraries, autosaves, backups, analysis outputs, and
manufacturing files out of the import. Point BOM exports to the existing
ignored production directory instead of a workstation-specific location.

Validation with KiCad 9.0.1:
- Netlist export succeeds and referenced custom libraries resolve.
- DRC: 0 errors, 40 warnings, 0 unconnected items, 0 schematic mismatches.
- ERC: 27 errors and 71 warnings, identical to the source design.

The pre-existing missing JTAG 3D model (87831-1420.stp) is not supplied by
the source project and remains unresolved.
Parts:
- removed TP4: TestPoint, TestPoint:TestPoint_Pad_D1.0mm, symbol Connector:TestPoint
- C45: renamed from C41; LCSC C90057 -> C90057
- C50: renamed from C46; value 1u -> 1n; LCSC C77386 -> C77026
- renumbered C36 to C40, C37 to C41, C38 to C42, C39 to C43, C40 to C44, C42 to C46, C43 to C47, C44 to C48, C45 to C49, TP3 to TP2
Connections:
- net +5V renamed +3.3VP
Other:
- moved on the sheet: C40, C41, C42, C43, C44, C45, C46, C47, C48, C49, C50, IC2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
