File: hardware/Power(VCC1V0M).kicad_sch (KiCad schematic)
At the start: 27 parts, among them IC1 LT3071, J2 SMA, J3 SMA

Commit message: Update hardware design and include board logo
Sync the saved schematics, PCB, project settings, and referenced custom
libraries with the updated design. Include the LOGO footprint and register
it in the project footprint table. The board now contains 524 footprints.

Keep unused source libraries, autosaves, backups, analysis outputs, and
manufacturing files out of the import. Point BOM exports to the existing
ignored production directory instead of a workstation-specific location.

Validation with KiCad 9.0.1:
- Netlist export succeeds and referenced custom libraries resolve.
- DRC: 0 errors, 40 warnings, 0 unconnected items, 0 schematic mismatches.
- ERC: 27 errors and 71 warnings, identical to the source design.

The pre-existing missing JTAG 3D model (87831-1420.stp) is not supplied by
the source project and remains unresolved.
Parts:
- removed TP2: TestPoint, TestPoint:TestPoint_Pad_D1.0mm, symbol Connector:TestPoint
- C31: renamed from C27; LCSC C77047 -> C85973
- C33: renamed from C29; footprint Capacitor_SMD:C_0603_1608Metric -> Capacitor_SMD:C_0805_2012Metric; LCSC C77047 -> C117966
- C34: renamed from C30; footprint Capacitor_SMD:C_0603_1608Metric -> Capacitor_SMD:C_0805_2012Metric; LCSC C90057 -> C408144
- C39: renamed from C35; value 1u -> 1n; LCSC C77386 -> C77026
- renumbered C23 to C27, C24 to C28, C25 to C29, C26 to C30, C28 to C32, C31 to C35, C32 to C36, C33 to C37, C34 to C38
Connections:
- net +5V renamed +3.3VP
