File: hardware/Power(VCC1V2C,VCC2V5,VCC2V8).kicad_sch (KiCad schematic)
At the start: 26 parts, among them IC3 MCP1727-ADJE_MF, IC4 MCP1727-ADJE_MF, IC5 MCP1727-ADJE_MF

Commit message: Update hardware design and include board logo
Sync the saved schematics, PCB, project settings, and referenced custom
libraries with the updated design. Include the LOGO footprint and register
it in the project footprint table. The board now contains 524 footprints.

Keep unused source libraries, autosaves, backups, analysis outputs, and
manufacturing files out of the import. Point BOM exports to the existing
ignored production directory instead of a workstation-specific location.

Validation with KiCad 9.0.1:
- Netlist export succeeds and referenced custom libraries resolve.
- DRC: 0 errors, 40 warnings, 0 unconnected items, 0 schematic mismatches.
- ERC: 27 errors and 71 warnings, identical to the source design.

The pre-existing missing JTAG 3D model (87831-1420.stp) is not supplied by
the source project and remains unresolved.
Parts:
- removed TP10, TP6, TP9: TestPoint, TestPoint:TestPoint_Pad_D1.0mm, symbol Connector:TestPoint
- added R23: 100k, Resistor_SMD:R_0603_1608Metric, symbol Device:R
- C51: renamed from C47; LCSC C90057 -> C90057
- C52: renamed from C48; LCSC C90057 -> C90057
- C53: renamed from C49; value 4700 pF -> 4.7n; LCSC C85973 -> C85980
- C54: renamed from C50; LCSC C90057 -> C90057
- C55: renamed from C51; LCSC C90057 -> C90057
- C56: renamed from C52; LCSC C90057 -> C90057
- C57: renamed from C53; value 4700 pF -> 4.7n; LCSC C85973 -> C85980
- C58: renamed from C54; LCSC C90057 -> C90057
- C59: renamed from C55; value 4700 pF -> 4.7n; LCSC C85973 -> C85980
- R25: renamed from R24; value 261k -> 357k; LCSC C2930083 -> C913223
- R26: renamed from R25; value 91k -> 357k; LCSC C2930083 -> C913223
- R30: renamed from R29; value 13k -> 51k
- renumbered R23 to R24, R26 to R27, R27 to R28, R28 to R29, TP5 to TP3, TP7 to TP4, TP8 to TP5
Connections:
- net +5V: now also R23.2
- net 1V8_DELAY: now also R23.1
Other:
- note added: "Ideal voltage is 3.3V 3.28V = 0.41V*((357000/51000)+1)"
- note removed: "Ideal voltage is 3.3V 3.28V = 0.41V*((261000/51000)+1)"
- moved on the sheet: C51, C53, R22, R24, TP3
