File: hardware/Power_root.kicad_sch (KiCad schematic)
At the start: 40 parts, among them J1 Jack-DC, U1 LT8625SPJV-1#TRMPBF, U2 LT8625SPJV-1#TRMPBF

Commit message: Update hardware design and include board logo
Sync the saved schematics, PCB, project settings, and referenced custom
libraries with the updated design. Include the LOGO footprint and register
it in the project footprint table. The board now contains 524 footprints.

Keep unused source libraries, autosaves, backups, analysis outputs, and
manufacturing files out of the import. Point BOM exports to the existing
ignored production directory instead of a workstation-specific location.

Validation with KiCad 9.0.1:
- Netlist export succeeds and referenced custom libraries resolve.
- DRC: 0 errors, 40 warnings, 0 unconnected items, 0 schematic mismatches.
- ERC: 27 errors and 71 warnings, identical to the source design.

The pre-existing missing JTAG 3D model (87831-1420.stp) is not supplied by
the source project and remains unresolved.
Parts:
- added C10, C22: 1u, Capacitor_SMD:C_0603_1608Metric, symbol Device:C
- added C25, C26: 1u, Capacitor_SMD:C_0603_1608Metric, symbol Device:C_Small
- added U3: TI LP2985-33DBVR, Package_TO_SOT_SMD:SOT-23-5, symbol Regulator_Linear:LP2985-3.3
- C1, C2: footprint Capacitor_SMD:C_1206_3216Metric -> Capacitor_SMD:C_1210_3225Metric; LCSC C77091 -> C309062
- C13: renamed from C12; footprint Capacitor_SMD:C_1206_3216Metric -> Capacitor_SMD:C_1210_3225Metric; LCSC C77091 -> C309062
- C14: renamed from C13; footprint Capacitor_SMD:C_1206_3216Metric -> Capacitor_SMD:C_1210_3225Metric; LCSC C77091 -> C309062
- C15: renamed from C14; footprint Capacitor_SMD:C_0603_1608Metric -> Capacitor_SMD:C_0805_2012Metric; LCSC C77386 -> C126592
- C16: renamed from C15; footprint Capacitor_SMD:C_1206_3216Metric -> Capacitor_SMD:C_1210_3225Metric; LCSC C91604 -> C21397
- C17: renamed from C16; footprint Capacitor_SMD:C_1206_3216Metric -> Capacitor_SMD:C_1210_3225Metric; LCSC C91604 -> C21397
- C18: renamed from C17; footprint Capacitor_SMD:C_1206_3216Metric -> Capacitor_SMD:C_1210_3225Metric; LCSC C91604 -> C21397
- C19: renamed from C18; footprint Capacitor_SMD:C_1206_3216Metric -> Capacitor_SMD:C_1210_3225Metric; LCSC C91604 -> C21397
- C20: renamed from C19; footprint Capacitor_SMD:C_1206_3216Metric -> Capacitor_SMD:C_1210_3225Metric; LCSC C91604 -> C21397
- C3: footprint Capacitor_SMD:C_0603_1608Metric -> Capacitor_SMD:C_0805_2012Metric; LCSC C77386 -> C126592
- C4, C5, C6, C7, C8: footprint Capacitor_SMD:C_1206_3216Metric -> Capacitor_SMD:C_1210_3225Metric; LCSC C91604 -> C21397
- R11: value 33.2k -> 49.9k; LCSC C185338 -> C705780
- R8: LCSC C861797 -> C861309
- R9: LCSC C705780 -> C2075328
- renumbered C10 to C11, C11 to C12, C20 to C21, C21 to C23, C22 to C24
Connections:
- net +5V: now also C25.1, U3.1 (VIN), U3.3 (ON/~{OFF})
- net GND: now also C10.2, C22.2, C25.2, C26.2, U3.2 (GND)
- net at U1.11 (INTVCC): now also C10.1
- net at U2.11 (INTVCC): now also C22.1
- new net +3.3VP: C26.1, U3.5 (VOUT)
- no-connect marks 11 -> 10
Other:
- moved on the sheet: C11, D1, R6
